Commit message: octomap changes

File: turtlebot3_description/urdf/turtlebot3_waffle_pi_2.urdf.xacro (robot description, xacro)
@@ -173,4 +173,17 @@
     </collision>
   </link>
+  <joint name="ti_mmwave_joint" type="fixed">
+    <parent link="base_link"/>
+    <child link="ti_mmwave"/>
+    <origin xyz="0.070 0 0.100" rpy="0 -0.0872 0"/>
+  </joint>
+  <link name="ti_mmwave">
+    <collision>
+      <origin xyz="0.005 0.011 0.013" rpy="0 0 0"/>
+      <geometry>
+        <box size="0.015 0.030 0.027"/>
+      </geometry>
+    </collision>
+  </link>
   <joint name="camera_joint" type="fixed">
     <origin xyz="0.073 -0.011 0.084" rpy="0 0 0"/>
