Commit message: update viz and xacro file

File: turtlebot3_description/urdf/turtlebot3_waffle_pi_2_rplidar.urdf.xacro (robot description, xacro)
@@ -163,5 +163,5 @@
     <parent link="base_link"/>
     <child link="base_points2"/>
-    <origin xyz="0.070 0 0.100" rpy="0 0 0"/>
+    <origin xyz="0.070 0 0.100" rpy="0 -0.0872 0"/>
   </joint>
   <link name="base_points2">

Commit message: add left side mounted radar link

File: turtlebot3_description/urdf/turtlebot3_waffle_pi_2_rplidar.urdf.xacro (robot description, xacro)
@@ -173,8 +173,21 @@
     </collision>
   </link>
-  <joint name="ti_mmwave_joint" type="fixed">
+  <!-- <joint name="ti_mmwave_joint" type="fixed">
     <parent link="base_link"/>
     <child link="ti_mmwave"/>
     <origin xyz="0.070 0 0.100" rpy="0 -0.0872 0"/>
+  </joint>
+  <link name="ti_mmwave">
+    <collision>
+      <origin xyz="0.005 0.011 0.013" rpy="0 0 0"/>
+      <geometry>
+        <box size="0.015 0.030 0.027"/>
+      </geometry>
+    </collision>
+  </link> -->
+  <joint name="ti_mmwave_joint" type="fixed">
+    <parent link="base_link"/>
+    <child link="ti_mmwave"/>
+    <origin xyz="-0.017 0.13 0.100" rpy="0 -0.0872 1.57"/>
   </joint>
   <link name="ti_mmwave">

Commit message: add new radar link in middle of bot

File: turtlebot3_description/urdf/turtlebot3_waffle_pi_2_rplidar.urdf.xacro (robot description, xacro)
@@ -173,4 +173,5 @@
     </collision>
   </link>
+  <!-- radar nach vorne vorne -->
   <!-- <joint name="ti_mmwave_joint" type="fixed">
     <parent link="base_link"/>
@@ -186,5 +187,20 @@
     </collision>
   </link> -->
+  <!-- radar nach vorne mitte -->
   <joint name="ti_mmwave_joint" type="fixed">
+    <parent link="base_link"/>
+    <child link="ti_mmwave"/>
+    <origin xyz="0.005 0 0.100" rpy="0 -0.0872 0"/>
+  </joint>
+  <link name="ti_mmwave">
+    <collision>
+      <origin xyz="0.005 0.011 0.013" rpy="0 0 0"/>
+      <geometry>
+        <box size="0.015 0.030 0.027"/>
+      </geometry>
+    </collision>
+  </link>
+  <!-- radar linke seite -->
+  <!-- <joint name="ti_mmwave_joint" type="fixed">
     <parent link="base_link"/>
     <child link="ti_mmwave"/>
@@ -198,5 +214,5 @@
       </geometry>
     </collision>
-  </link>
+  </link> -->
   <joint name="camera_joint" type="fixed">
     <origin xyz="0.073 -0.011 0.084" rpy="0 0 0"/>

Commit message: change external camera to fisheye

File: turtlebot3_description/urdf/turtlebot3_waffle_pi_2_rplidar.urdf.xacro (robot description, xacro)
@@ -130,5 +130,5 @@
     <parent link="base_link"/>
     <child link="imu_link"/>
-    <origin xyz="0.0 -0.02 0.068" rpy="0 0 0"/>
+    <origin xyz="0.0 -0.03 0.103" rpy="0 0 0"/>
   </joint>
   <link name="imu_link"/>
@@ -136,5 +136,5 @@
     <parent link="base_link"/>
     <child link="base_scan"/>
-    <origin xyz="-0.095 -0.002 0.122" rpy="0 0 0"/>
+    <origin xyz="-0.095 -0.002 0.157" rpy="0 0 0"/>
   </joint>
   <link name="base_scan">
@@ -163,5 +163,5 @@
     <parent link="base_link"/>
     <child link="base_points2"/>
-    <origin xyz="0.070 0 0.100" rpy="0 -0.0872 0"/>
+    <origin xyz="0.070 0 0.135" rpy="0 -0.0872 0"/>
   </joint>
   <link name="base_points2">
@@ -191,5 +191,5 @@
     <parent link="base_link"/>
     <child link="ti_mmwave"/>
-    <origin xyz="0.005 0 0.100" rpy="0 -0.0872 0"/>
+    <origin xyz="0.005 0 0.135" rpy="0 -0.0872 0"/>
   </joint>
   <link name="ti_mmwave">
@@ -216,5 +216,5 @@
   </link> -->
   <joint name="camera_joint" type="fixed">
-    <origin xyz="0.073 -0.011 0.084" rpy="0 0 0"/>
+    <origin xyz="0.06 0.07 0.095" rpy="0 0 0"/>
     <parent link="base_link"/>
     <child link="camera_link"/>
@@ -228,5 +228,5 @@
     </collision>
   </link>
-  <joint name="camera_rgb_joint" type="fixed">
+  <!-- <joint name="camera_rgb_joint" type="fixed">
     <origin xyz="0.003 0.011 0.009" rpy="0 0 0"/>
     <parent link="camera_link"/>
@@ -239,4 +239,17 @@
     <child link="camera_rgb_optical_frame"/>
   </joint>
-  <link name="camera_rgb_optical_frame"/>
+  <link name="camera_rgb_optical_frame"/> -->
+  <joint name="fisheye_camera_joint" type="fixed">
+    <origin xyz="0.06 -0.08 0.1" rpy="0 0 0"/>
+    <parent link="base_link"/>
+    <child link="fisheye_camera_link"/>
+  </joint>
+  <link name="fisheye_camera_link">
+    <collision>
+      <origin xyz="0.005 0.011 0.013" rpy="0 0 0"/>
+      <geometry>
+        <box size="0.015 0.030 0.027"/>
+      </geometry>
+    </collision>
+  </link>
 </robot>

Commit message: add new radar pose

File: turtlebot3_description/urdf/turtlebot3_waffle_pi_2_rplidar.urdf.xacro (robot description, xacro)
@@ -188,5 +188,5 @@
   </link> -->
   <!-- radar nach vorne mitte -->
-  <joint name="ti_mmwave_joint" type="fixed">
+  <!-- <joint name="ti_mmwave_joint" type="fixed">
     <parent link="base_link"/>
     <child link="ti_mmwave"/>
@@ -200,5 +200,5 @@
       </geometry>
     </collision>
-  </link>
+  </link> -->
   <!-- radar linke seite -->
   <!-- <joint name="ti_mmwave_joint" type="fixed">
@@ -215,4 +215,18 @@
     </collision>
   </link> -->
+  <!-- radar nach vorne mitte gedreht 10grad links -->
+  <joint name="ti_mmwave_joint" type="fixed">
+    <parent link="base_link"/>
+    <child link="ti_mmwave"/>
+    <origin xyz="0.006 0 0.135" rpy="0 -0.0872 0.1745"/>
+  </joint>
+  <link name="ti_mmwave">
+    <collision>
+      <origin xyz="0.005 0.011 0.013" rpy="0 0 0"/>
+      <geometry>
+        <box size="0.015 0.030 0.027"/>
+      </geometry>
+    </collision>
+  </link>
   <joint name="camera_joint" type="fixed">
     <origin xyz="0.06 0.07 0.095" rpy="0 0 0"/>

Commit message: add image transformation node

File: turtlebot3_description/urdf/turtlebot3_waffle_pi_2_rplidar.urdf.xacro (robot description, xacro)
@@ -261,7 +261,21 @@
   <link name="fisheye_camera_link">
     <collision>
-      <origin xyz="0.005 0.011 0.013" rpy="0 0 0"/>
-      <geometry>
-        <box size="0.015 0.030 0.027"/>
+      <origin xyz="0.005 0.005 0.005" rpy="0 0 0"/>
+      <geometry>
+        <box size="0.01 0.01 0.01"/>
+      </geometry>
+    </collision>
+  </link>
+  <joint name="fisheye_camera_rviz_image_joint" type="fixed">
+    <!-- <origin xyz="0.06 -0.08 -0.1" rpy="-1.5708 0 -1.5708"/> -->
+    <origin xyz="0.209 0 -0.11" rpy="3.14159 0 -1.5707"/>
+    <parent link="fisheye_camera_link"/>
+    <child link="fisheye_camera_rviz_image_link"/>
+  </joint>
+  <link name="fisheye_camera_rviz_image_link">
+    <collision>
+      <origin xyz="0.1 0.2 0.3" rpy="0 0 0"/>
+      <geometry>
+        <box size="0 0 0"/>
       </geometry>
     </collision>

Commit message: update xacro file radar position

File: turtlebot3_description/urdf/turtlebot3_waffle_pi_2_rplidar.urdf.xacro (robot description, xacro)
@@ -188,5 +188,5 @@
   </link> -->
   <!-- radar nach vorne mitte -->
-  <!-- <joint name="ti_mmwave_joint" type="fixed">
+  <joint name="ti_mmwave_joint" type="fixed">
     <parent link="base_link"/>
     <child link="ti_mmwave"/>
@@ -200,5 +200,5 @@
       </geometry>
     </collision>
-  </link> -->
+  </link>
   <!-- radar linke seite -->
   <!-- <joint name="ti_mmwave_joint" type="fixed">
@@ -216,5 +216,5 @@
   </link> -->
   <!-- radar nach vorne mitte gedreht 10grad links -->
-  <joint name="ti_mmwave_joint" type="fixed">
+  <!-- <joint name="ti_mmwave_joint" type="fixed">
     <parent link="base_link"/>
     <child link="ti_mmwave"/>
@@ -228,5 +228,5 @@
       </geometry>
     </collision>
-  </link>
+  </link> -->
   <joint name="camera_joint" type="fixed">
     <origin xyz="0.06 0.07 0.095" rpy="0 0 0"/>

Commit message: update links and joints

File: turtlebot3_description/urdf/turtlebot3_waffle_pi_2_rplidar.urdf.xacro (robot description, xacro)
@@ -255,5 +255,5 @@
   <link name="camera_rgb_optical_frame"/> -->
   <joint name="fisheye_camera_joint" type="fixed">
-    <origin xyz="0.06 -0.08 0.1" rpy="0 0 0"/>
+    <origin xyz="0.06 -0.035 0.1" rpy="0 0 0"/>
     <parent link="base_link"/>
     <child link="fisheye_camera_link"/>
@@ -269,5 +269,5 @@
   <joint name="fisheye_camera_rviz_image_joint" type="fixed">
     <!-- <origin xyz="0.06 -0.08 -0.1" rpy="-1.5708 0 -1.5708"/> -->
-    <origin xyz="0.209 0 -0.11" rpy="3.14159 0 -1.5707"/>
+    <origin xyz="0.342 0 -0.11" rpy="3.14159 0 -1.5707"/> <!-- x = 0.342 = 608px height / 2 + 38mm abstand-->
     <parent link="fisheye_camera_link"/>
     <child link="fisheye_camera_rviz_image_link"/>

Commit message: update

File: turtlebot3_description/urdf/turtlebot3_waffle_pi_2_rplidar.urdf.xacro (robot description, xacro)
@@ -230,5 +230,5 @@
   </link> -->
   <joint name="camera_joint" type="fixed">
-    <origin xyz="0.06 0.07 0.095" rpy="0 0 0"/>
+    <origin xyz="0.08 0.07 0.095" rpy="0 0 0"/>
     <parent link="base_link"/>
     <child link="camera_link"/>

Commit message: add fisheye device specifier; 10degree radar

File: turtlebot3_description/urdf/turtlebot3_waffle_pi_2_rplidar.urdf.xacro (robot description, xacro)
@@ -188,5 +188,5 @@
   </link> -->
   <!-- radar nach vorne mitte -->
-  <joint name="ti_mmwave_joint" type="fixed">
+  <!-- <joint name="ti_mmwave_joint" type="fixed">
     <parent link="base_link"/>
     <child link="ti_mmwave"/>
@@ -200,5 +200,5 @@
       </geometry>
     </collision>
-  </link>
+  </link> -->
   <!-- radar linke seite -->
   <!-- <joint name="ti_mmwave_joint" type="fixed">
@@ -216,5 +216,5 @@
   </link> -->
   <!-- radar nach vorne mitte gedreht 10grad links -->
-  <!-- <joint name="ti_mmwave_joint" type="fixed">
+  <joint name="ti_mmwave_joint" type="fixed">
     <parent link="base_link"/>
     <child link="ti_mmwave"/>
@@ -228,5 +228,5 @@
       </geometry>
     </collision>
-  </link> -->
+  </link>
   <joint name="camera_joint" type="fixed">
     <origin xyz="0.08 0.07 0.095" rpy="0 0 0"/>

Commit message: update recordbag script; update rviz; update full launch; update xacro 15grad

File: turtlebot3_description/urdf/turtlebot3_waffle_pi_2_rplidar.urdf.xacro (robot description, xacro)
@@ -216,8 +216,22 @@
   </link> -->
   <!-- radar nach vorne mitte gedreht 10grad links -->
+  <!-- <joint name="ti_mmwave_joint" type="fixed">
+    <parent link="base_link"/>
+    <child link="ti_mmwave"/>
+    <origin xyz="0.006 0 0.135" rpy="0 -0.0872 0.1745"/>
+  </joint>
+  <link name="ti_mmwave">
+    <collision>
+      <origin xyz="0.005 0.011 0.013" rpy="0 0 0"/>
+      <geometry>
+        <box size="0.015 0.030 0.027"/>
+      </geometry>
+    </collision>
+  </link> -->
+  <!-- radar nach vorne mitte gedreht 15grad links -->
   <joint name="ti_mmwave_joint" type="fixed">
     <parent link="base_link"/>
     <child link="ti_mmwave"/>
-    <origin xyz="0.006 0 0.135" rpy="0 -0.0872 0.1745"/>
+    <origin xyz="0.006 0 0.135" rpy="0 -0.0872 0.2618"/>
   </joint>
   <link name="ti_mmwave">
